Commit message: Update URDF and hardware interface for IMeta Y1 robot, including mesh adjustments and improved joint configurations

File: imeta_y1_description/urdf/imeta_y1/imeta_y1_macro.urdf.xacro (robot description, xacro)
@@ -16,5 +16,5 @@
       </inertial>
       <visual>
-        <origin xyz="0 0 0.067" rpy="0 0 1.5707963" />
+        <origin xyz="0 0 0" rpy="0 0 0" />
         <geometry>
           <mesh filename="package://imeta_y1_description/meshes/imeta_y1/base_link.STL" />
@@ -25,5 +25,5 @@
       </visual>
       <collision>
-        <origin xyz="0 0 0.067" rpy="0 0 1.5707963" />
+        <origin xyz="0 0 0" rpy="0 0 0" />
         <geometry>
           <mesh filename="package://imeta_y1_description/meshes/imeta_y1/base_link.STL" />
@@ -54,9 +54,9 @@
     </link>
     <joint name="joint1" type="revolute">
-      <origin xyz="0 0 0.067" rpy="0 0 0" />
+      <origin xyz="0 0 0.06675" rpy="0 0 0" />
       <parent link="${root_link}" />
       <child link="link1" />
-      <axis xyz="0 0 -1" />
-      <limit lower="-3.0" upper="3.0" effort="30" velocity="5" />
+      <axis xyz="0 0 1" />
+      <limit lower="-3.0" upper="3.0" effort="30" velocity="10" />
     </joint>
     <link name="link2">
@@ -87,5 +87,5 @@
       <child link="link2" />
       <axis xyz="0 0 1" />
-      <limit lower="-3.5" upper="0.2" effort="100" velocity="5" />
+      <limit lower="-3.5" upper="0.2" effort="120" velocity="10" />
     </joint>
     <link name="link3">
@@ -116,5 +116,5 @@
       <child link="link3" />
       <axis xyz="0 0 1" />
-      <limit lower="-0.2" upper="4.1" effort="30" velocity="5" />
+      <limit lower="-0.2" upper="3.25" effort="30" velocity="10" />
     </joint>
     <link name="link4">
@@ -145,5 +145,5 @@
       <child link="link4" />
       <axis xyz="0 0 1" />
-      <limit lower="-2.5" upper="1.7" effort="10" velocity="20" />
+      <limit lower="-2.35" upper="1.6" effort="30" velocity="10" />
     </joint>
     <link name="link5">
@@ -174,34 +174,34 @@
       <child link="link5" />
       <axis xyz="0 0 1" />
-      <limit lower="-2.0" upper="2.0" effort="10" velocity="20" />
+      <limit lower="-1.6" upper="1.6" effort="20" velocity="30" />
     </joint>
     <link name="link6">
-      <!-- <inertial>
-        <origin xyz="-0.006 0.000 0.047" rpy="0 0 0" />
-        <mass value=" 0.479" />
-        <inertia ixx="0.000" ixy="0.000" ixz=" 0.000" iyy="0.001" iyz="0.000" izz="0.001" />
-      </inertial>
-      <visual>
-        <origin xyz="0 0 0" rpy="0 0 0" />
-        <geometry>
-          <mesh filename="package://imeta_y1_description/meshes/imeta_y1/Link6.STL" />
-        </geometry>
-        <material name="">
-          <color rgba="1 1 1 1" />
-        </material>
-      </visual>
-      <collision>
-        <origin xyz="0 0 0" rpy="0 0 0" />
-        <geometry>
-          <mesh filename="package://imeta_y1_description/meshes/imeta_y1/Link6.STL" />
-        </geometry>
-      </collision> -->
+    <inertial>
+      <origin xyz="0.031920 -0.000193 0.043758" rpy="0 0 0" />
+      <mass value="0.150000" />
+      <inertia ixx="0.000058" ixy="0.000000" ixz="0.000000" iyy="0.000027" iyz="0.000000" izz="0.000027" />
+    </inertial>
+    <visual>
+      <origin xyz="0 0 0" rpy="0 0 0" />
+      <geometry>
+        <mesh filename="package://imeta_y1_description/meshes/imeta_y1/Link6.STL" />
+      </geometry>
+      <material name="">
+        <color rgba="1 1 1 1" />
+      </material>
+    </visual>
+    <collision>
+      <origin xyz="0 0 0" rpy="0 0 0" />
+      <geometry>
+        <mesh filename="package://imeta_y1_description/meshes/imeta_y1/Link6.STL" />
+      </geometry>
+    </collision>
     </link>
     <joint name="joint6" type="revolute">
-      <origin xyz="0.0235 0 0.044" rpy="3.1416 1.5708 3.1416" />
+      <origin xyz="0.0235 0 0.0440000000000001" rpy="-3.14159265330655 0 0" />
       <parent link="link5" />
       <child link="link6" />
-      <axis xyz="0 0 1" />
-      <limit lower="-3.0" upper="3.0" effort="10" velocity="20" />
+      <axis xyz="1 0 0" />
+      <limit lower="-2.75" upper="2.75" effort="20" velocity="30" />
     </joint>
   </xacro:macro>

File: imeta_y1_description/urdf/imeta_y1/include/real_world.ros2_control.xacro (robot description, xacro)
@@ -5,5 +5,4 @@
         <plugin>imeta_y1_hardware/IMetaY1HW</plugin>
         <param name="can_interface">can0</param>
-        <param name="urdf_path">package://imeta_y1_description/urdf/imeta_y1.urdf</param>
         <!-- 0: only arm, 1: gripper_T, 2: gripper_G, 3: gripper_GT -->
         <param name="arm_end_type">0</param>
